File: pcb_comms/gps.kicad_sch (KiCad schematic)
At the start: 0 parts

Commit message: Add usb and gps
Parts:
- added BT1: COIN_Cell, symbol Device:Battery_Cell
- added C42: 47pF, symbol Device:C
- added C43: 1.0uF, symbol Device:C
- added CR3: SD1206S040S1R0, SD1206_AVX, symbol SCHOTTKY_DIODE_SD1206S040S1R0:SD1206S040S1R0
- added D1: PESD0402-240, DIONC1005X43N, symbol ESD_PROTECTION_DIODE_PESD0402-240:PESD0402-240
- added FB1: 2.66ohm, symbol Device:FerriteBead_Small
- added J3: Conn_Coaxial, symbol Connector:Conn_Coaxial
- added JP1: Open, symbol Jumper:SolderJumper_3_Open
- added R10, R11, R12, R13, R5, R6, R7, R8, R9: 33, symbol Device:R
- added R14, R15: 2.2k, symbol Device:R
- added R16: 3.3k, symbol Device:R
- added U1: MAX-M10M-00B, MOD18_MAX-M10M_UBL, symbol GPS_MAX_M10S:MAX-M10M-00B
Connections:
- new net: D1.2, FB1.1, J3.1 (In), U1.11 (RF_IN)
- new net: C42.1, FB1.2, R5.1
- new net: CR3.1, R16.1
- new net: JP1.1 (A), R14.2
- new net: JP1.3 (B), R15.2
- new net +3V3: CR3.2, JP1.2 (C), U1.7 (V_IO), U1.8 (VCC)
- new net GND: BT1.2 (-), C42.2, C43.2, D1.1, J3.2 (Ext), U1.1 (GND), U1.10 (GND), U1.12 (GND)
- new net INT: R11.2
- new net MAX_BACKUP: BT1.1 (+), C43.1, R16.2, U1.6 (V_BCKP)
- new net MAX_INT: R11.1, U1.5 (EXTINT)
- new net MAX_PPS: R12.1, U1.4 (TIMEPULSE)
- new net MAX_RESET_N: R6.1, U1.9 (RESET_N)
- new net MAX_RXI: R8.1, U1.3 (RXD)
- new net MAX_SAFE_N: R13.1, U1.18 (SAFEBOOT_N)
- new net MAX_SCL: R10.1, U1.17 (SCL)
- new net MAX_SDA: R9.1, U1.16 (SDA)
- new net MAX_TXO: R7.1, U1.2 (TXD)
- new net PPS: R12.2
- new net RESET_N: R6.2
- new net RXI: R8.2
- new net SAFE_N: R13.2
- new net SCL: R10.2, R14.1
- new net SDA: R15.1, R9.2
- new net TXO: R7.2
- new net VCC_RF: R5.2, U1.14 (VCC_RF)
- no-connect marks 0 -> 2
Other:
- note added: "RTC BACKUP"
