File: pcb_comms/antenna_deploy.kicad_sch (KiCad schematic)
At the start: 6 parts, among them Q2 PMOS, Q3 NMOS

Commit message: Last update
Other:
- company: (none) -> Sanie Peralta, Alejandro Campo
- title: (none) -> PC1: APRS & GPS
Changed lines of the file:
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@@
 	(generator_version "9.0")
 	(paper "A4")
+	(title_block
+		(title "PC1: APRS & GPS")
+		(date "2026-04-01")
+		(rev "1.0")
+		(company "Sanie Peralta, Alejandro Campo")
+		(comment 1 "Introducción a la Ingeniería Satelital ")
+		(comment 2 "Primer Parcial")
+	)
 	(junction
 		(at 88.9 57.15)
