File: pcb_comms/mcu.kicad_sch (KiCad schematic)
At the start: 25 parts, among them U2 STM32WLE5CCU6, Y1 G43270018, Y3 32MHz

Commit message: Update schematic
Parts:
- removed C4, C5: 0.1uF, Capacitor_SMD:C_0805_2012Metric_Pad1.18x1.45mm_HandSolder, symbol Device:C
Connections:
- net +3V3: now also U2.11 (VDD); no longer C10.1, C11.1, C32.1, L2.1, U2.47 (VLXSMPS)
- net AUX0: no longer names the net of U2.6 (PB8)
- net AUX1: no longer names the net of U2.13 (PA5)
- net AUX2: no longer names the net of U2.14 (PA6)
- net AUX3: no longer names the net of U2.15 (PA7)
- net AUX4: no longer names the net of U2.16 (PA8)
- net AUX5: no longer names the net of U2.17 (PA9)
- new net VDDRF: C32.1
- new net VLXSMPS: C10.1, C11.1, L2.1, U2.47 (VLXSMPS)
- no-connect marks 3 -> 9
Other:
- moved on the sheet: C32, C33, C34, C6, C7, FB2

Commit message: re arrange
Parts:
- removed Y1: G43270018, CRYSTAL_32.687KHz_G43270018:CRYSTAL_32.687KHz_G43270018, symbol CRYSTAL_32.687KHz_G43270018:G43270018
- C33: footprint Capacitor_SMD:C_0805_2012Metric_Pad1.18x1.45mm_HandSolder -> Capacitor_SMD:C_0603_1608Metric_Pad1.08x0.95mm_HandSolder
Connections:
- net VDDRF is gone; now on net +3V3: C32.1
- net +3V3: now also FB2.1; no longer FB2.2, U2.37 (VBAT)
- net RF_CRL_TO_STM32: now also U2.17 (PA9); no longer U2.12 (PA4)
- net VDDA: now also FB2.2; no longer FB2.1
- net OSC_RTC_IN: no longer names the net of U2.39 (PC14-OSC32_IN)
- net OSC_RTC_OUT: no longer names the net of U2.40 (PC15-OSC32_OUT)
- no-connect marks 9 -> 11
Other:
- note removed: "RTC"
- moved on the sheet: C32, FB2

Commit message: PCB v2
Connections:
- net DRA_SQ_TO_STM32: now also U2.16 (PA8); no longer U2.31 (PB2)
- net STM32_TO_DRA_ENA: now also U2.14 (PA6); no longer U2.32 (PB12)
- net STM32_TO_DRA_PTT: now also U2.15 (PA7); no longer U2.30 (PB0-VDD_TCXO)
- no-connect marks 11 -> 8
Changed lines of the file:
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@@
-	)
-	(no_connect
-		(at 167.64 132.08)
 	)
 	(no_connect
@@
 	)
 	(no_connect
-		(at 167.64 129.54)
-	)
-	(no_connect
 		(at 167.64 127)
-	)
-	(no_connect
-		(at 167.64 134.62)
 	)
 	(no_connect
@@
 	(wire
 		(pts
+			(xy 152.4 132.08) (xy 167.64 132.08)
+		)
+		(stroke
+			(width 0)
+			(type default)
+		)
+	)
+	(wire
+		(pts
 			(xy 238.76 157.48) (xy 254 157.48)
 		)
@@
 	(wire
 		(pts
-			(xy 238.76 142.24) (xy 257.81 142.24)
-		)
-		(stroke
-			(width 0)
-			(type default)
-		)
-	)
-	(wire
-		(pts
 			(xy 123.19 38.1) (xy 123.19 41.91)
 		)
@@
 	(wire
 		(pts
-			(xy 238.76 144.78) (xy 257.81 144.78)
-		)
-		(stroke
-			(width 0)
-			(type default)
-		)
-	)
-	(wire
-		(pts
 			(xy 25.4 46.99) (xy 25.4 36.83)
 		)
@@
 	(wire
 		(pts
+			(xy 152.4 129.54) (xy 167.64 129.54)
+		)
+		(stroke
+			(width 0)
+			(type default)
+		)
+	)
+	(wire
+		(pts
 			(xy 238.76 137.16) (xy 257.81 137.16)
 		)
@@
 	(wire
 		(pts
-			(xy 238.76 139.7) (xy 257.81 139.7)
-		)
-		(stroke
-			(width 0)
-			(type default)
-		)
-	)
-	(wire
-		(pts
 			(xy 271.78 149.86) (xy 275.59 149.86)
 		)
@@
 		(pts
 			(xy 45.72 161.29) (xy 58.42 161.29)
+		)
+		(stroke
+			(width 0)
+			(type default)
+		)
+	)
+	(wire
+		(pts
+			(xy 152.4 134.62) (xy 167.64 134.62)
 		)
 		(stroke
@@
 	(global_label "DRA_SQ_TO_STM32"
 		(shape input)
-		(at 257.81 142.24 0)
-		(effects
-			(font
-				(size 1.27 1.27)
-			)
-			(justify left)
-		)
-		(property "Intersheetrefs" "${INTERSHEET_REFS}"
-			(at 279.4822 129.54 0)
-			(effects
-				(font
-					(size 1.27 1.27)
-				)
-				(justify left)
+		(at 152.4 134.62 180)
+		(effects
+			(font
+				(size 1.27 1.27)
+			)
+			(justify right)
+		)
+		(property "Intersheetrefs" "${INTERSHEET_REFS}"
+			(at 130.7278 121.92 0)
+			(effects
+				(font
+					(size 1.27 1.27)
+				)
+				(justify right)
 				(hide yes)
 			)
@@
 	(global_label "STM32_TO_DRA_PTT"
 		(shape input)
-		(at 257.81 144.78 0)
+		(at 152.4 132.08 180)
 		(fields_autoplaced yes)
 		(effects
@@
 				(size 1.27 1.27)
 			)
-			(justify left)
-		)
-		(property "Intersheetrefs" "${INTERSHEET_REFS}"
-			(at 278.8774 144.78 0)
-			(effects
-				(font
-					(size 1.27 1.27)
-				)
-				(justify left)
+			(justify right)
+		)
+		(property "Intersheetrefs" "${INTERSHEET_REFS}"
+			(at 131.3326 132.08 0)
+			(effects
+				(font
+					(size 1.27 1.27)
+				)
+				(justify right)
 				(hide yes)
 			)
@@
 	(global_label "STM32_TO_DRA_ENA"
 		(shape input)
-		(at 257.81 139.7 0)
+		(at 152.4 129.54 180)
 		(fields_autoplaced yes)
 		(effects
@@
 				(size 1.27 1.27)
 			)
-			(justify left)
-		)
-		(property "Intersheetrefs" "${INTERSHEET_REFS}"
-			(at 279.2403 139.7 0)
-			(effects
-				(font
-					(size 1.27 1.27)
-				)
-				(justify left)
-				(hide yes)
-			)
+			(justify right)
+		)
+		(property "Intersheetrefs" "${INTERSHEET_REFS}"
+			(at 130.9697 129.54 0)
+			(effects
+				(font
+					(size 1.27 1.27)
+				)
+				(justify right)
+				(hide yes)
+			)

Commit message: PCB v2.1
Parts:
- C1, C10, C11, C14, C16, C2, C26, C3, C31, C32, C34, C6, C7: footprint Capacitor_SMD:C_0805_2012Metric_Pad1.18x1.45mm_HandSolder -> Capacitor_SMD:C_0603_1608Metric_Pad1.08x0.95mm_HandSolder
Connections:
- no-connect marks 8 -> 12
Other:
- note removed: "Capactiores cerca del STM32"
- moved on the sheet: C32, C33, C34, U2

Commit message: Add STM32 gps test 1
Other:
- note removed: "VDDRF Capacitors"
- company: Sanie Peralta, Alejandro Campo -> Sanie Peralta
- title: PC1: APRS & GPS -> PAYLOAD 1: APRS
- moved on the sheet: C1, C2, C3, C6, C7, FB2
