File: pcb_comms/aprs_radio.kicad_sch (KiCad schematic)
At the start: 33 parts, among them J4 SMA_CONNECTOR, Q1 DTC144EET1G, U3 DRA818V

Commit message: Add STM32 gps test 1
Other:
- company: Sanie Peralta, Alejandro Campo -> Sanie Peralta
- title: PC1: APRS & GPS -> PAYLOAD 1: APRS
Changed lines of the file:
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@@
 	(paper "A4")
 	(title_block
-		(title "PC1: APRS & GPS")
+		(title "PAYLOAD 1: APRS")
 		(date "2026-04-01")
-		(rev "1.0")
-		(company "Sanie Peralta, Alejandro Campo")
+		(rev "1.1")
+		(company "Sanie Peralta")
 		(comment 1 "Introducción a la Ingeniería Satelital ")
-		(comment 2 "Primer Parcial")
 	)
 	(text "AF_OUT"
