File: pcb_comms/pcb_comms_board.kicad_pcb (KiCad board)
At the start: 4 copper layers, 90 x 90.2 mm, 102 parts, among them IC1 LDL1117S33R, IC2 TPS2553QDBVRQ1, IC4 BGS12WN6E6329XTSA1, J1 Conn_01x06_Pin, J2 Conn_02x20_Odd_Even, J4 SMA_CONNECTOR, J6 SMA_CONNECTOR, J7 USB-B-Micro, J9 GPS, Q1 DTC144EET1G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

Commit message: PCB v2
Parts:
- moved CR2 52.3 mm to (140.0, 72.0), turned to 90 degrees
- moved J1 45.1 mm to (145.1, 72.5), turned to 180 degrees
- moved SB3 38.7 mm to (150.2, 68.6), turned to 90 degrees
- moved R1 31.9 mm to (176.9, 99.4), turned to -90 degrees
- moved D3 27.9 mm to (168.0, 99.5), turned to -90 degrees
- moved C12 25.6 mm to (165.2, 99.6), turned to -90 degrees
- moved S1 22.7 mm to (181.3, 99.0)
- moved C43 9.37 mm to (116.5, 101.8)
- moved L10 4.34 mm to (113.9, 94.9)
- moved C45 4.31 mm to (116.0, 94.8)
- moved C49 4.29 mm to (120.3, 94.8)
- moved C46 4.28 mm to (118.1, 94.8)
- moved R8 4.06 mm to (120.4, 101.8)
- moved C9 3.94 mm to (138.0, 60.2)
- moved IC2 3.94 mm to (133.2, 61.1)
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Connections:
- FB2 pad 1: /MCU/VDDA -> +3V3
- FB2 pad 2: +3V3 -> /MCU/VDDA
- U2 pad 14: unconnected-(U2-PA6-Pad14) -> STM32_TO_DRA_ENA
- U2 pad 15: unconnected-(U2-PA7-Pad15) -> STM32_TO_DRA_PTT
- U2 pad 16: unconnected-(U2-PA8-Pad16) -> DRA_SQ_TO_STM32
- U2 pad 30: STM32_TO_DRA_PTT -> unconnected-(U2-PB0-VDD_TCXO-Pad30)
- U2 pad 31: DRA_SQ_TO_STM32 -> unconnected-(U2-PB2-Pad31)
- U2 pad 32: STM32_TO_DRA_ENA -> unconnected-(U2-PB12-Pad32)
Routing:
- net +3V3: track 68.7 -> 273.4 mm, vias 4 -> 15
- net DRA_TO_STM32_ADC: track 10.6 -> 160.0 mm, vias 0 -> 2
- net STM32_DAC_TO_DRA: track 0.00 -> 112.0 mm, vias 0 -> 2
- net GND: track 72.9 -> 161.6 mm, vias 176 -> 226
- net DRA_SQ_TO_STM32: track 0.00 -> 76.7 mm, vias 0 -> 2
- net DRA_TX_UART1_RX: track 0.00 -> 75.4 mm, vias 0 -> 2
- net DRA_RX_UART1_TX: track 0.00 -> 73.6 mm, vias 0 -> 2
- net STM32_TO_DRA_PTT: track 2.19 -> 69.3 mm, vias 0 -> 2
- net UART_RX: track 0.00 -> 59.9 mm, vias 0 -> 2
- net UART2_TX: track 0.00 -> 56.5 mm
- net STM32_TO_DRA_ENA: track 7.51 -> 62.1 mm, vias 0 -> 2
- net OCP_EN: track 1.69 -> 40.2 mm
- net OCP_NFAULT: track 1.21 -> 37.5 mm
- net /MCU/STM32_BOOT: track 13.1 -> 48.8 mm
- net STM32_NRST: track 33.4 -> 66.7 mm, vias 2 -> 3
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
Commit message: PCB v2.1
Parts:
- C1, C10, C11, C14, C16, C17, C2, C21, C22, C24, C26, C28, C29, C3, C31, C32, C34, C6, C7: footprint Capacitor_SMD:C_0805_2012Metric_Pad1.18x1.45mm_HandSolder -> Capacitor_SMD:C_0603_1608Metric_Pad1.08x0.95mm_HandSolder
- C9: footprint Capacitor_SMD:C_1210_3225Metric_Pad1.33x2.70mm_HandSolder -> Capacitor_SMD:C_Elec_6.3x7.7
- J1: footprint Connector_PinHeader_2.54mm:PinHeader_1x06_P2.54mm_Vertical_SMD_Pin1Right -> CONN_01x06_87898-0666:CONN_01x06_87898-0666
- L1, L10, L9: footprint Inductor_SMD:L_0805_2012Metric_Pad1.05x1.20mm_HandSolder -> Inductor_SMD:L_1210_3225Metric_Pad1.42x2.65mm_HandSolder
- R12: value 100 -> 100R
- moved C12 24.1 mm to (147.9, 82.8)
- moved D3 24.0 mm to (150.7, 82.9)
- moved R14 21.6 mm to (117.4, 61.1)
- moved R10 19.3 mm to (114.0, 62.9)
- moved IC2 19.3 mm to (113.9, 59.6)
- moved C8 19.3 mm to (107.9, 59.7)
- moved C47 17.7 mm to (136.4, 82.6), turned to 0 degrees
- moved C9 14.3 mm to (123.8, 60.4), turned to 0 degrees
- moved CR2 9.65 mm to (135.7, 63.4), turned to 0 degrees
- moved IC1 8.27 mm to (130.7, 79.9), turned to 90 degrees
- moved R9 4.73 mm to (117.1, 71.7)
- moved FB2 4.45 mm to (166.8, 57.9), turned to 0 degrees
- moved C48 3.02 mm to (118.3, 68.6), turned to -90 degrees
- moved J1 2.53 mm to (143.0, 71.1), turned to -90 degrees
- moved D6 2.46 mm to (115.8, 68.6), turned to 90 degrees
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Routing:
- net +3V3: track 273.4 -> 332.7 mm, vias 15 -> 6
- net STM32_NRST: track 66.7 -> 30.5 mm, vias 3 -> 2
- net OCP_NFAULT: track 37.5 -> 61.7 mm
- net OCP_EN: track 40.2 -> 57.5 mm
- net /APRS_RADIO/3V3_DRA: track 119.5 -> 131.7 mm, vias 3 -> 2
- net VBAT_IN: track 20.7 -> 31.2 mm
- net GND: track 161.6 -> 154.5 mm, vias 226 -> 237
- net Net-(J1-Pin_6): track 9.49 -> 16.3 mm, vias 0 -> 2
- net Net-(J1-Pin_4): track 4.27 -> 11.0 mm
- net UART_RX: track 59.9 -> 54.3 mm
- net DRA_TO_STM32_ADC: track 160.0 -> 164.5 mm
- net RF_CRL_TO_STM32: track 28.7 -> 32.8 mm, vias 0 -> 2
- net /MCU/VDDA: track 10.7 -> 14.6 mm
- net /OCP/ILIM: track 6.19 -> 2.45 mm
- net /MCU/VDDRF1V55: track 40.1 -> 36.8 mm, vias 0 -> 2
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
Commit message: PCB v2.2
Routing:
- net OCP_EN: track 57.5 -> 56.1 mm
- net DRA_SQ_TO_STM32: track 77.4 -> 76.6 mm
- net GND: track 154.5 -> 154.2 mm, vias 237 -> 247

Commit message: Add STM32 gps test 1
Parts:
- added G***: LOGO, logos:fiuna, F.Cu at (167.1, 108.1)
- added G***: LOGO, logos:sat, F.Cu at (170.3, 125.4)
- GPS: renamed from J9; value GPS -> CONN_GPS
- L5: footprint Inductor_SMD:L_0402_1005Metric_Pad0.77x0.64mm_HandSolder -> Inductor_SMD:L_0603_1608Metric_Pad1.05x0.95mm_HandSolder
- L6: footprint Inductor_SMD:L_0402_1005Metric_Pad0.77x0.64mm_HandSolder -> Resistor_SMD:R_0603_1608Metric_Pad0.98x0.95mm_HandSolder
- moved SMA2 28.3 mm to (182.6, 114.5)
- moved C28 5.40 mm to (177.6, 86.1)
- moved L7 2.21 mm to (175.9, 89.3), turned to -90 degrees
- moved SMA1 0.97 mm to (183.9, 85.3)
- moved L6 0.88 mm to (165.2, 80.1)
- moved C3 0.79 mm to (162.6, 61.9)
- moved C9 0.76 mm to (124.5, 60.5)
- moved FB2 0.75 mm to (167.1, 58.6)
- moved L5 0.72 mm to (173.4, 83.2)
- moved L3 0.66 mm to (168.1, 81.4)
- moved C15 0.66 mm to (168.1, 79.4)
- moved C44 0.59 mm to (117.8, 116.9)
- moved C22 0.56 mm to (173.3, 84.8)
- moved C37 0.54 mm to (120.2, 116.9)
- moved R14 0.25 mm to (117.2, 61.0)
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- renumbered U3 to DRA818V, J1 to JTAG, J6 to SMA1, J4 to SMA2, U2 to STM, J7 to USB
Routing:
- net /APRS_RADIO/DRA_ANT: track 9.76 -> 37.7 mm
- net DRA_TX_UART1_RX: track 76.2 -> 61.3 mm
- net DRA_RX_UART1_TX: track 74.2 -> 60.8 mm
- net DRA_TO_STM32_ADC: track 164.5 -> 177.5 mm
- net STM32_DAC_TO_DRA: track 109.3 -> 120.7 mm
- net GND: track 154.2 -> 146.3 mm, vias 247 -> 271
- net STM32_TO_DRA_PTT: track 70.1 -> 76.4 mm
- net JTCK_SWCLK_TO_STM32: track 28.2 -> 21.9 mm
- net STM32_TO_DRA_ENA: track 63.4 -> 57.7 mm
- net +3V3: track 332.7 -> 329.5 mm
- net /APRS_RADIO/3V3_DRA: track 131.7 -> 130.0 mm
- net DRA_SQ_TO_STM32: track 76.6 -> 78.2 mm
- net /MCU/VDDRF1V55: track 36.8 -> 38.2 mm
- net /RF/RFIN2: track 5.82 -> 4.71 mm
- net /RF/SMA1: track 11.2 -> 10.1 mm
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Other:
- board text added: "CR1"
- board text added: "CR2"
- board text added: "PAYLOAD 1: APRS DIGIPEATER"
