File: pcb_comms/pcb_comms_board.kicad_sch (KiCad schematic)
At the start: 4 parts

Commit message: Update route
Parts:
- H1, H2, H3, H4: footprint MountingHole:MountingHole_3.2mm_M3_Pad_Via -> MountingHole:MountingHole_3.2mm_M3_DIN965_Pad_TopBottom
Changed lines of the file:
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@@
 			)
 		)
-		(property "Footprint" "MountingHole:MountingHole_3.2mm_M3_Pad_Via"
+		(property "Footprint" "MountingHole:MountingHole_3.2mm_M3_DIN965_Pad_TopBottom"
 			(at 39.37 66.04 0)
 			(effects
@@
 			)
 		)
-		(property "Footprint" "MountingHole:MountingHole_3.2mm_M3_Pad_Via"
+		(property "Footprint" "MountingHole:MountingHole_3.2mm_M3_DIN965_Pad_TopBottom"
 			(at 57.15 66.04 0)
 			(effects
@@
 			)
 		)
-		(property "Footprint" "MountingHole:MountingHole_3.2mm_M3_Pad_Via"
+		(property "Footprint" "MountingHole:MountingHole_3.2mm_M3_DIN965_Pad_TopBottom"
 			(at 48.26 66.04 0)
 			(effects
@@
 			)
 		)
-		(property "Footprint" "MountingHole:MountingHole_3.2mm_M3_Pad_Via"
+		(property "Footprint" "MountingHole:MountingHole_3.2mm_M3_DIN965_Pad_TopBottom"
 			(at 66.04 66.04 0)
 			(effects

Commit message: Add STM32 gps test 1
Other:
- company: Sanie Peralta, Alejandro Campo -> Sanie Peralta
- title: PC1: APRS & GPS -> PAYLOAD 1: APRS
Changed lines of the file:
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@@
 	(paper "A4")
 	(title_block
-		(title "PC1: APRS & GPS")
+		(title "PAYLOAD 1: APRS")
 		(date "2026-04-01")
-		(rev "1.0")
-		(company "Sanie Peralta, Alejandro Campo")
+		(rev "1.1")
+		(company "Sanie Peralta")
 		(comment 1 "Introducción a la Ingeniería Satelital ")
-		(comment 2 "Primer Parcial")
 	)
 	(symbol
